File: electrical/scheme/digitizer.kicad_pcb (KiCad board)
At the start: 2 copper layers, 0 parts

Commit message: a
Parts:
- added C1: 100n, Capacitors_SMD:C_0805_HandSoldering, F.Cu at (67.3, 77.5)
- added C10, C11, C12, C13, C16, C20, C7, C8, C9: 4u7, Capacitors_SMD:C_0805_HandSoldering, F.Cu at (148.5, 105.0)
- added C14, C18, C19, C22, C23, C24, C25, C26, C28, C29, C30, C31, C34, C35, C36, C38, C42, C43, C48, C49, C54, C55, C60, C61, C64, C65, C66, C67, C70, C71, C72, C73, C74, C75, C78, C79, C80, C81, C82, C83: 100n, Capacitors_SMD:C_0805_HandSoldering, F.Cu at (148.5, 105.0)
- added C15, C32, C33, C68, C69, C76, C77: 1n, Capacitors_SMD:C_0805_HandSoldering, F.Cu at (148.5, 105.0)
- added C17: 3n, Capacitors_SMD:C_0805_HandSoldering, F.Cu at (148.5, 105.0)
- added C2: 18p, Capacitors_SMD:C_0805_HandSoldering, F.Cu at (68.6, 83.8)
- added C21, C37: 2n2, Capacitors_SMD:C_0805_HandSoldering, F.Cu at (148.5, 105.0)
- added C27: 330u, Capacitors_ThroughHole:C_Radial_D10_L20_P5, F.Cu at (195.6, 111.8)
- added C3: 18p, Capacitors_SMD:C_0805_HandSoldering, F.Cu at (69.8, 88.9)
- added C39: 330u, Capacitors_ThroughHole:C_Radial_D10_L20_P5, F.Cu at (175.3, 106.7)
- added C4: 100n, Capacitors_SMD:C_0805_HandSoldering, F.Cu at (69.8, 92.7)
- added C40, C46, C52, C58: 3u3, Capacitors_SMD:C_0805_HandSoldering, F.Cu at (148.5, 105.0)
- added C41, C45, C47, C51, C53, C57, C59, C63: 22n, Capacitors_SMD:C_0805_HandSoldering, F.Cu at (148.5, 105.0)
- added C44, C50, C56, C62: 120n, Capacitors_SMD:C_0805_HandSoldering, F.Cu at (148.5, 105.0)
- added C5: 100n, Capacitors_SMD:C_0805_HandSoldering, F.Cu at (69.8, 97.8)
- added C6: 4u7, Capacitors_SMD:C_0805_HandSoldering, F.Cu at (71.1, 102.9)
- added D1: LED, LEDs:LED-3MM, F.Cu at (120.7, 105.4)
- added D2: LED, LEDs:LED-3MM, F.Cu at (157.5, 87.6)
- added D3: 1n5819, Diodes_ThroughHole:Diode_DO-41_SOD81_Horizontal_RM10, F.Cu at (177.8, 120.7)
- added D4: 1n5819, Diodes_ThroughHole:Diode_DO-41_SOD81_Horizontal_RM10, F.Cu at (195.6, 127.0)
- added L1: 50uH, my-lib:my_inductance, F.Cu at (188.0, 97.8)
- added L2: 50uH, my-lib:my_inductance, F.Cu at (167.6, 96.5)
- added P1: mode, Pin_Headers:Pin_Header_Straight_1x02, F.Cu at (87.6, 87.6)
- added P10: in-2, Sockets_BNC:BNC_Socket_TYCO-AMP_LargePads, F.Cu at (91.4, 73.7)
- added P11: in-3, Sockets_BNC:BNC_Socket_TYCO-AMP_LargePads, F.Cu at (228.6, 76.2)
- added P12: in-1, Sockets_BNC:BNC_Socket_TYCO-AMP_LargePads, F.Cu at (254.0, 76.2)
- added P2: ~rst~, Pin_Headers:Pin_Header_Straight_1x01, F.Cu at (148.5, 105.0)
- added P3: ext, Socket_Strips:Socket_Strip_Angled_1x13, F.Cu at (87.6, 129.5)
- added P4: trig, Sockets_BNC:BNC_Socket_TYCO-AMP_LargePads, F.Cu at (193.0, 78.7)
- added P5: trig-mode, Pin_Headers:Pin_Header_Angled_1x03, F.Cu at (158.8, 137.2)
- added P6: swd, Socket_Strips:Socket_Strip_Angled_1x03, F.Cu at (138.4, 135.9)
- added P7: out-0, Sockets_BNC:BNC_Socket_TYCO-AMP_LargePads, F.Cu at (167.6, 73.7)
- added P8: out-1, Sockets_BNC:BNC_Socket_TYCO-AMP_LargePads, F.Cu at (143.5, 73.7)
- added P9: in-0, Sockets_BNC:BNC_Socket_TYCO-AMP_LargePads, F.Cu at (116.8, 73.7)
- added R1, R10, R11, R19, R20, R25, R39, R4, R6, R7, R8: 10k 5%, Resistors_SMD:R_0805_HandSoldering, F.Cu at (148.5, 105.0)
- added R12, R13: 10k, Resistors_SMD:R_0805_HandSoldering, F.Cu at (148.5, 105.0)
- added R14: 0, Resistors_SMD:R_0805_HandSoldering, F.Cu at (148.5, 105.0)
- added R15: 50 5%, Resistors_SMD:R_0805_HandSoldering, F.Cu at (148.5, 105.0)
- added R16, R38: 0.15 5%, Resistors_SMD:R_0805_HandSoldering, F.Cu at (148.5, 105.0)
- added R17, R42: 1k1 1%, Resistors_SMD:R_0805_HandSoldering, F.Cu at (148.5, 105.0)
- added R18: 1k5 5%, Resistors_SMD:R_0805_HandSoldering, F.Cu at (148.5, 105.0)
- added R2, R3, R9: 1k 5%, Resistors_SMD:R_0805_HandSoldering, F.Cu at (148.5, 105.0)
- added R21, R23: 8k2 5%, Resistors_SMD:R_0805_HandSoldering, F.Cu at (148.5, 105.0)
- added R22, R24: 1 5%, Resistors_SMD:R_0805_HandSoldering, F.Cu at (148.5, 105.0)
- added R26: 13k 5%, Resistors_SMD:R_0805_HandSoldering, F.Cu at (148.5, 105.0)
- added R27, R28, R29, R30, R31, R32, R45, R46, R51, R52, R57, R58, R63, R64, R67, R68, R69, R70, R71, R72, R73, R74: 16 5%, Resistors_SMD:R_0805_HandSoldering, F.Cu at (148.5, 105.0)
- added R33: 120k 5%, Resistors_SMD:R_0805_HandSoldering, F.Cu at (148.5, 105.0)
- added R34, R36: 1k6 5%, Resistors_SMD:R_0805_HandSoldering, F.Cu at (148.5, 105.0)
- added R35, R37: 3k3 5%, Resistors_SMD:R_0805_HandSoldering, F.Cu at (148.5, 105.0)
- added R40, R41: 12k 5%, Resistors_SMD:R_0805_HandSoldering, F.Cu at (148.5, 105.0)
- added R43, R49, R55, R61: 806 1%, Resistors_SMD:R_0805_HandSoldering, F.Cu at (148.5, 105.0)
- added R44, R50, R56, R62: 1k91 1%, Resistors_SMD:R_0805_HandSoldering, F.Cu at (148.5, 105.0)
- added R47, R53, R59, R65: 9k31 1%, Resistors_SMD:R_0805_HandSoldering, F.Cu at (148.5, 105.0)
- added R48, R54, R60, R66: 21k 1%, Resistors_SMD:R_0805_HandSoldering, F.Cu at (148.5, 105.0)
- added R5: 100 5%, Resistors_SMD:R_0805_HandSoldering, F.Cu at (148.5, 105.0)
- added U1: AD8672, Housings_SOIC:SOIC-8_3.9x4.9mm_Pitch1.27mm, F.Cu at (125.7, 94.0)
- added U10: crystal-4pin, crystal-smd-5x3:CRYSTAL-SMD-5x3, F.Cu at (158.8, 104.1)
- added U100: AD8672, Housings_SOIC:SOIC-8_3.9x4.9mm_Pitch1.27mm, F.Cu at (151.1, 88.9)
- added U101: AD8672, Housings_SOIC:SOIC-8_3.9x4.9mm_Pitch1.27mm, F.Cu at (111.8, 87.6)
- added U11: CP2102, my-lib:CP2102, F.Cu at (133.3, 104.1)
- added U12: MINI-USB-B, my-lib:my-mini-usb-b, F.Cu at (110.5, 99.1)
- added U13: BAT54S, Housings_SOT-23_SOT-143_TSOT-6:SOT-23, F.Cu at (148.5, 105.0)
- added U14, U15, U16: MCP1703T-3302E/CB, Housings_SOT-23_SOT-143_TSOT-6:SOT-23, F.Cu at (148.5, 105.0)
- added U17: AD7683, Housings_SSOP:MSOP-8_3x3mm_Pitch0.65mm, F.Cu at (119.4, 99.1)
- added U18: NCP3063, Housings_SOIC:SOIC-8_3.9x4.9mm_Pitch1.27mm, F.Cu at (129.5, 121.9)
- added U19: ADG5204, Housings_SSOP:TSSOP-14_4.4x5mm_Pitch0.65mm, F.Cu at (82.5, 101.6)
- added U2: AD8672, Housings_SOIC:SOIC-8_3.9x4.9mm_Pitch1.27mm, F.Cu at (129.5, 87.6)
- added U20: NCP3063, Housings_SOIC:SOIC-8_3.9x4.9mm_Pitch1.27mm, F.Cu at (86.4, 116.8)
- added U21: AD5543, Housings_SOIC:SOIC-8_3.9x4.9mm_Pitch1.27mm, F.Cu at (127.0, 113.0)
- added U22: AD5543, Housings_SOIC:SOIC-8_3.9x4.9mm_Pitch1.27mm, F.Cu at (109.2, 119.4)
- added U23: AD5543, Housings_SOIC:SOIC-8_3.9x4.9mm_Pitch1.27mm, F.Cu at (101.6, 110.5)
- added U24: AD5543, Housings_SOIC:SOIC-8_3.9x4.9mm_Pitch1.27mm, F.Cu at (142.2, 90.2)
- added U3: AD8672, Housings_SOIC:SOIC-8_3.9x4.9mm_Pitch1.27mm, F.Cu at (139.7, 96.5)
- added U4: AD8672, Housings_SOIC:SOIC-8_3.9x4.9mm_Pitch1.27mm, F.Cu at (153.7, 96.5)
- added U5: AD8672, Housings_SOIC:SOIC-8_3.9x4.9mm_Pitch1.27mm, F.Cu at (162.6, 109.2)
- added U6: AD8672, Housings_SOIC:SOIC-8_3.9x4.9mm_Pitch1.27mm, F.Cu at (161.3, 118.1)
- added U7: AD8672, Housings_SOIC:SOIC-8_3.9x4.9mm_Pitch1.27mm, F.Cu at (167.6, 127.0)
- added U8: AD8672, Housings_SOIC:SOIC-8_3.9x4.9mm_Pitch1.27mm, F.Cu at (143.5, 121.9)
- added U9: AD8672, Housings_SOIC:SOIC-8_3.9x4.9mm_Pitch1.27mm, F.Cu at (153.7, 123.2)
- added stm321: STM32F103CBT6, my-lib:LQFP48, F.Cu at (115.6, 113.0)

Commit message: a
Parts:
- removed U12: MINI-USB-B, my-lib:my-mini-usb-b
- added P13: USB_B, Connect:USB_B, F.Cu at (55.9, 49.2)
- moved R5 129.4 mm to (27.9, 57.9)
- moved R2 127.7 mm to (26.9, 66.0)
- moved C71 123.6 mm to (28.7, 74.4)
- moved C70 121.6 mm to (28.2, 87.6)
- moved C76 121.4 mm to (34.8, 62.5)
- moved C69 121.3 mm to (27.7, 94.2)
- moved C68 120.3 mm to (29.0, 118.6)
- moved C63 119.6 mm to (31.5, 129.5)
- moved C52 119.3 mm to (29.3, 102.0)
- moved C60 119.3 mm to (31.5, 81.9)
- moved C61 117.9 mm to (36.1, 69.6)
- moved C51 116.7 mm to (32.1, 113.8)
- moved C77 116.6 mm to (43.2, 54.9)
- moved C57 116.6 mm to (35.4, 76.8)
- moved C43 115.3 mm to (34.5, 87.8)
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Connections:
- U11 pad 11: Net-(U11-Pad11) -> (no net)
- U11 pad 2: Net-(U11-Pad2) -> (no net)
- U11 pad 27: Net-(U11-Pad27) -> (no net)
- U11 pad 28: Net-(U11-Pad28) -> (no net)
- U18 pad 8: Net-(U18-Pad8) -> (no net)
- U20 pad 8: Net-(U20-Pad8) -> (no net)
- stm321 pad 17: /adc-mosi -> (no net)
- stm321 pad 27: /dac-miso -> (no net)
- stm321 pad 38: Net-(stm321-Pad38) -> (no net)
- stm321 pad 39: Net-(stm321-Pad39) -> (no net)
- stm321 pad 40: Net-(stm321-Pad40) -> (no net)

Commit message: a
Parts:
- added C84: 1n, Capacitors_SMD:C_0805_HandSoldering, F.Cu at (-5.08, -8.89)
- added C85: 680u, Capacitors_ThroughHole:C_Radial_D10_L20_P5, F.Cu at (-5.08, -26.7)
- added C86: 1n, Capacitors_SMD:C_0805_HandSoldering, F.Cu at (-11.4, -3.81)
- added C87: 680u, Capacitors_ThroughHole:C_Radial_D10_L20_P5, F.Cu at (19.1, -22.9)
- added C88: 1n, Capacitors_SMD:C_0805_HandSoldering, F.Cu at (-24.1, 0.00)
- added C89: 680u, Capacitors_ThroughHole:C_Radial_D10_L20_P5, F.Cu at (3.81, -8.89)
- added C90: 1n, Capacitors_SMD:C_0805_HandSoldering, F.Cu at (-8.89, 3.81)
- added C91: 680u, Capacitors_ThroughHole:C_Radial_D10_L20_P5, F.Cu at (6.35, -24.1)
- added L3: 100uH, my-lib:my_inductance, F.Cu at (-17.8, 10.2)
- added L4: 100uH, my-lib:my_inductance, F.Cu at (-20.3, -11.4)
- added L5: 100uH, my-lib:my_inductance, F.Cu at (-12.7, -22.9)
- added L6: 100uH, my-lib:my_inductance, F.Cu at (-38.1, 2.54)
- C27, C39: value 330u -> 680u
- L1: value 50uH -> 100uH
- P1: footprint Pin_Headers:Pin_Header_Straight_1x02 -> Pin_Headers:Pin_Header_Angled_1x02
- P6: footprint Socket_Strips:Socket_Strip_Angled_1x03 -> Socket_Strips:Socket_Strip_Straight_1x03
- moved C27 221.9 mm to (35.6, -41.9)
- moved C39 190.3 mm to (20.3, -3.81)
- moved L1 188.6 mm to (41.9, -21.6)
- moved C10 164.9 mm to (79.7, -62.3)
- moved C11 164.9 mm to (91.2, -72.6)
- moved C12 164.9 mm to (122.5, -77.4)
- moved C13 164.9 mm to (96.5, -38.8)
- moved C14 164.9 mm to (108.8, -51.6)
- moved C15 164.9 mm to (98.7, -51.7)
- moved C16 164.9 mm to (104.6, -84.1)
- moved C17 164.9 mm to (118.0, -54.5)
- moved C18 164.9 mm to (81.7, -69.0)
- moved C19 164.9 mm to (88.7, -62.9)
- moved C2 164.9 mm to (96.5, -78.7)
- moved C20 164.9 mm to (78.1, -84.9)
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Connections:
- C23 pad 1: /dac-v-0/v+ -> Net-(C23-Pad1)
- C27 pad 1: /dac-v-0/v+ -> Net-(C23-Pad1)
- C37 pad 2: /dac-v-0/v- -> Net-(C37-Pad2)
- C38 pad 1: /dac-v-0/v- -> Net-(C37-Pad2)
- C39 pad 1: /dac-v-0/v- -> GND
- C39 pad 2: GND -> Net-(C37-Pad2)
- D3 pad 1: /dac-v-0/v+ -> Net-(C23-Pad1)
- D4 pad 2: /dac-v-0/v- -> Net-(C37-Pad2)
- R42 pad 1: /dac-v-0/v- -> Net-(C37-Pad2)
- U20 pad 4: /dac-v-0/v- -> Net-(C37-Pad2)

Commit message: a
Parts:
- added C92: 100n, Capacitors_SMD:C_0805_HandSoldering, F.Cu at (108.4, 71.2)
- added C93: 100n, Capacitors_SMD:C_0805_HandSoldering, F.Cu at (117.8, 83.6)
- added C94: 100n, Capacitors_SMD:C_0805_HandSoldering, F.Cu at (107.0, 82.2)
- added C95: 100n, Capacitors_SMD:C_0805_HandSoldering, F.Cu at (121.2, 74.0)
- added C96: 4u7, Capacitors_SMD:C_0805_HandSoldering, F.Cu at (106.0, 71.2)
- added C97, C98: 4u7, Capacitors_SMD:C_0805_HandSoldering, F.Cu at (0.00, 0.00)
- added L7: 47uH, Capacitors_SMD:C_1206_HandSoldering, F.Cu at (-1.27, 11.4)
- added L8: 47uH, Capacitors_SMD:C_1206_HandSoldering, F.Cu at (22.9, 33.2)
- R10, R8: value 10k 5% -> 33k 5%
- moved R5 193.4 mm to (121.8, 77.2)
- moved C2 164.4 mm to (126.4, 82.9)
- moved U13 154.7 mm to (143.6, 61.9), turned to 180 degrees
- moved C3 150.9 mm to (126.4, 74.5)
- moved U10 149.8 mm to (126.1, 78.6), turned to 270 degrees
- moved C10 145.1 mm to (55.2, 80.7), turned to 270 degrees
- moved C4 142.6 mm to (123.0, 70.5)
- moved U16 135.4 mm to (58.0, 80.6)
- moved R6 129.9 mm to (110.7, 62.8)
- moved R7 128.8 mm to (123.1, 68.4), turned to 180 degrees
- moved C13 127.8 mm to (58.6, 83.2), turned to 180 degrees
- moved C8 117.9 mm to (43.1, 66.1), turned to 270 degrees
- moved R8 116.8 mm to (139.8, 61.8), turned to 270 degrees
- moved R9 97.1 mm to (156.8, 64.5), turned to 90 degrees
- moved R10 96.2 mm to (147.1, 61.9), turned to 90 degrees
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Connections:
- C11 pad 1: /dac-v-0/dac-ref -> Net-(C11-Pad1)
- C12 pad 1: /adc-ref -> Net-(C12-Pad1)
- U14 pad 2: /dac-v-0/dac-ref -> Net-(C11-Pad1)
- U15 pad 2: /adc-ref -> Net-(C12-Pad1)

Commit message: a
Parts:
- removed U15: MCP1703T-3302E/CB, Housings_SOT-23_SOT-143_TSOT-6:SOT-23
- added U12: ref196, Housings_SOIC:SOIC-8_3.9x4.9mm_Pitch1.27mm, F.Cu at (-45.5, 124.3)
- L2: value 50uH -> 100uH
- L3, L4, L5, L6: value 100uH -> 47uH; footprint my-lib:my_inductance -> Capacitors_SMD:C_1206_HandSoldering
- U14: value MCP1703T-3302E/CB -> ref196; footprint Housings_SOT-23_SOT-143_TSOT-6:SOT-23 -> Housings_SOIC:SOIC-8_3.9x4.9mm_Pitch1.27mm
- moved D4 356.9 mm to (-123.0, 49.9), turned to 270 degrees
- moved D3 346.8 mm to (-64.0, 176.1), turned to 90 degrees
- moved R17 338.5 mm to (-55.5, 178.2), turned to 270 degrees
- moved L2 331.6 mm to (-116.9, 44.9), turned to 270 degrees
- moved R16 324.1 mm to (-49.0, 171.3)
- moved R19 323.7 mm to (-53.3, 178.2), turned to 90 degrees
- moved U18 301.9 mm to (-56.4, 172.4)
- moved C21 287.9 mm to (-61.3, 174.6), turned to 270 degrees
- moved C18 275.5 mm to (-49.1, 173.5)
- moved R39 267.4 mm to (-113.6, 60.1), turned to 90 degrees
- moved R38 264.6 mm to (-109.9, 51.3), turned to 90 degrees
- moved R42 263.9 mm to (-117.3, 60.1), turned to 270 degrees
- moved C23 263.2 mm to (-66.8, 172.6), turned to 90 degrees
- moved U20 250.1 mm to (-115.2, 53.8)
- moved C12 245.6 mm to (-37.4, 109.0), turned to 270 degrees
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Connections:
- U14 pad 1: GND -> (no net)
- U14 pad 2: Net-(C11-Pad1) -> /Vbus
- U14 pad 3: /Vbus -> VDD
