File: electrical/scheme/dac-v.sch (KiCad schematic (older format))
At the start: 13 parts, among them U21 AD5543, U22 AD5543, U8 AD8672

Commit message: a
Changed lines of the file:
@@
 AR Path="/55A0A529/55A0AE22" Ref="U21"  Part="1"
 AR Path="/55A5B809/55A0AE22" Ref="U23"  Part="1"
-F 0 "U23" H 8400 7900 60  0000 C CNN
+F 0 "U21" H 8400 7900 60  0000 C CNN
 F 1 "AD5543" H 8500 8350 60  0000 C CNN
 F 2 "Housings_SOIC:SOIC-8_3.9x4.9mm_Pitch1.27mm" H 7650 8100 60  0001 C CNN
@@
 AR Path="/55A0A529/55A0AE2F" Ref="C64"  Part="1"
 AR Path="/55A5B809/55A0AE2F" Ref="C72"  Part="1"
-F 0 "C72" H 7325 7550 50  0000 L CNN
+F 0 "C64" H 7325 7550 50  0000 L CNN
 F 1 "100n" H 7325 7350 50  0000 L CNN
 F 2 "Capacitors_SMD:C_0805_HandSoldering" H 7338 7300 30  0001 C CNN
@@
 AR Path="/55A0A529/55A0AE38" Ref="#PWR0159"  Part="1"
 AR Path="/55A5B809/55A0AE38" Ref="#PWR0173"  Part="1"
-F 0 "#PWR0173" H 7600 7450 30  0001 C CNN
+F 0 "#PWR0159" H 7600 7450 30  0001 C CNN
 F 1 "VDD" H 7600 7460 30  0000 C CNN
 F 2 "" H 7600 7350 60  0000 C CNN
@@
 AR Path="/55A0A529/55A0AE3F" Ref="U8"  Part="2"
 AR Path="/55A5B809/55A0AE3F" Ref="U9"  Part="2"
-F 0 "U9" H 9750 8100 60  0000 C CNN
+F 0 "U8" H 9750 8100 60  0000 C CNN
 F 1 "AD8672" H 9750 8500 60  0000 C CNN
 F 2 "Housings_SOIC:SOIC-8_3.9x4.9mm_Pitch1.27mm" H 9450 8300 60  0001 C CNN
@@
 AR Path="/55A0A529/55A0AE49" Ref="#PWR0160"  Part="1"
 AR Path="/55A5B809/55A0AE49" Ref="#PWR0174"  Part="1"
-F 0 "#PWR0174" H 8850 8350 50  0001 C CNN
+F 0 "#PWR0160" H 8850 8350 50  0001 C CNN
 F 1 "GNDA" H 8850 8450 50  0000 C CNN
 F 2 "" H 8850 8600 60  0000 C CNN
@@
 AR Path="/55A0A529/55A0AE5A" Ref="C68"  Part="1"
 AR Path="/55A5B809/55A0AE5A" Ref="C76"  Part="1"
-F 0 "C76" H 8825 7900 50  0000 L CNN
+F 0 "C68" H 8825 7900 50  0000 L CNN
 F 1 "1n" H 8825 7700 50  0000 L CNN
 F 2 "Capacitors_SMD:C_0805_HandSoldering" H 8838 7650 30  0001 C CNN
@@
 AR Path="/55A0A529/55A0AE9E" Ref="C65"  Part="1"
 AR Path="/55A5B809/55A0AE9E" Ref="C73"  Part="1"
-F 0 "C73" H 7525 6600 50  0000 L CNN
+F 0 "C65" H 7525 6600 50  0000 L CNN
 F 1 "100n" H 7525 6400 50  0000 L CNN
 F 2 "Capacitors_SMD:C_0805_HandSoldering" H 7538 6350 30  0001 C CNN
@@
 AR Path="/55A0A529/55A0AEA9" Ref="#PWR0161"  Part="1"
 AR Path="/55A5B809/55A0AEA9" Ref="#PWR0175"  Part="1"
-F 0 "#PWR0175" H 7150 6450 50  0001 C CNN
+F 0 "#PWR0161" H 7150 6450 50  0001 C CNN
 F 1 "GNDA" H 7150 6550 50  0000 C CNN
 F 2 "" H 7150 6700 60  0000 C CNN
@@
 AR Path="/55A0A529/55A0AEAF" Ref="#PWR0162"  Part="1"
 AR Path="/55A5B809/55A0AEAF" Ref="#PWR0176"  Part="1"
-F 0 "#PWR0176" H 7050 7300 50  0001 C CNN
+F 0 "#PWR0162" H 7050 7300 50  0001 C CNN
 F 1 "GND" H 7050 7400 50  0000 C CNN
 F 2 "" H 7050 7550 60  0000 C CNN
@@
 AR Path="/55A0A529/55A0B77B" Ref="U22"  Part="1"
 AR Path="/55A5B809/55A0B77B" Ref="U24"  Part="1"
-F 0 "U24" H 8700 3600 60  0000 C CNN
+F 0 "U22" H 8700 3600 60  0000 C CNN
 F 1 "AD5543" H 8800 4050 60  0000 C CNN
 F 2 "Housings_SOIC:SOIC-8_3.9x4.9mm_Pitch1.27mm" H 7950 3800 60  0001 C CNN
@@
 AR Path="/55A0A529/55A0B787" Ref="C66"  Part="1"
 AR Path="/55A5B809/55A0B787" Ref="C74"  Part="1"
-F 0 "C74" H 7625 3250 50  0000 L CNN
+F 0 "C66" H 7625 3250 50  0000 L CNN
 F 1 "100n" H 7625 3050 50  0000 L CNN
 F 2 "Capacitors_SMD:C_0805_HandSoldering" H 7638 3000 30  0001 C CNN
@@
 AR Path="/55A0A529/55A0B78F" Ref="#PWR0163"  Part="1"
 AR Path="/55A5B809/55A0B78F" Ref="#PWR0177"  Part="1"
-F 0 "#PWR0177" H 7900 3150 30  0001 C CNN
+F 0 "#PWR0163" H 7900 3150 30  0001 C CNN
 F 1 "VDD" H 7900 3160 30  0000 C CNN
 F 2 "" H 7900 3050 60  0000 C CNN
@@
 AR Path="/55A0A529/55A0B796" Ref="U8"  Part="1"
 AR Path="/55A5B809/55A0B796" Ref="U9"  Part="1"
-F 0 "U9" H 10050 3800 60  0000 C CNN
+F 0 "U8" H 10050 3800 60  0000 C CNN
 F 1 "AD8672" H 10050 4200 60  0000 C CNN
 F 2 "Housings_SOIC:SOIC-8_3.9x4.9mm_Pitch1.27mm" H 9750 4000 60  0001 C CNN
@@
 AR Path="/55A0A529/55A0B79F" Ref="#PWR0164"  Part="1"
 AR Path="/55A5B809/55A0B79F" Ref="#PWR0178"  Part="1"
-F 0 "#PWR0178" H 9150 4050 50  0001 C CNN
+F 0 "#PWR0164" H 9150 4050 50  0001 C CNN
 F 1 "GNDA" H 9150 4150 50  0000 C CNN
 F 2 "" H 9150 4300 60  0000 C CNN
@@
 AR Path="/55A0A529/55A0B7B0" Ref="C69"  Part="1"
 AR Path="/55A5B809/55A0B7B0" Ref="C77"  Part="1"
-F 0 "C77" H 9125 3600 50  0000 L CNN
+F 0 "C69" H 9125 3600 50  0000 L CNN
 F 1 "1n" H 9125 3400 50  0000 L CNN
 F 2 "Capacitors_SMD:C_0805_HandSoldering" H 9138 3350 30  0001 C CNN
@@
 AR Path="/55A0A529/55A0B7BC" Ref="R67"  Part="1"
 AR Path="/55A5B809/55A0B7BC" Ref="R69"  Part="1"
-F 0 "R69" V 9780 3100 50  0000 C CNN
+F 0 "R67" V 9780 3100 50  0000 C CNN
 F 1 "16 5%" V 9700 3100 50  0000 C CNN
 F 2 "Resistors_SMD:R_0805_HandSoldering" V 9630 3100 30  0001 C CNN
@@
 AR Path="/55A0A529/55A0B7C2" Ref="C70"  Part="1"
 AR Path="/55A5B809/55A0B7C2" Ref="C78"  Part="1"
-F 0 "C78" H 9975 3450 50  0000 L CNN
+F 0 "C70" H 9975 3450 50  0000 L CNN
 F 1 "100n" H 9975 3250 50  0000 L CNN
 F 2 "Capacitors_SMD:C_0805_HandSoldering" H 9988 3200 30  0001 C CNN
@@
 AR Path="/55A0A529/55A0B7CC" Ref="#PWR0165"  Part="1"
 AR Path="/55A5B809/55A0B7CC" Ref="#PWR0179"  Part="1"
-F 0 "#PWR0179" H 10200 3200 50  0001 C CNN
+F 0 "#PWR0165" H 10200 3200 50  0001 C CNN
 F 1 "GNDA" H 10200 3300 50  0000 C CNN
 F 2 "" H 10200 3450 60  0000 C CNN
@@
 AR Path="/55A0A529/55A0B7D5" Ref="R68"  Part="1"
 AR Path="/55A5B809/55A0B7D5" Ref="R70"  Part="1"
-F 0 "R70" V 9780 4800 50  0000 C CNN
+F 0 "R68" V 9780 4800 50  0000 C CNN
 F 1 "16 5%" V 9700 4800 50  0000 C CNN
 F 2 "Resistors_SMD:R_0805_HandSoldering" V 9630 4800 30  0001 C CNN
@@
 AR Path="/55A0A529/55A0B7E0" Ref="C71"  Part="1"
 AR Path="/55A5B809/55A0B7E0" Ref="C79"  Part="1"
-F 0 "C79" H 10025 4900 50  0000 L CNN
+F 0 "C71" H 10025 4900 50  0000 L CNN
 F 1 "100n" H 10025 4700 50  0000 L CNN
 F 2 "Capacitors_SMD:C_0805_HandSoldering" H 10038 4650 30  0001 C CNN
@@
 AR Path="/55A0A529/55A0B7E7" Ref="#PWR0166"  Part="1"
 AR Path="/55A5B809/55A0B7E7" Ref="#PWR0180"  Part="1"
-F 0 "#PWR0180" H 10000 4850 50  0001 C CNN
+F 0 "#PWR0166" H 10000 4850 50  0001 C CNN
 F 1 "GNDA" H 10000 4950 50  0000 C CNN
 F 2 "" H 10000 5100 60  0000 C CNN
@@
 AR Path="/55A0A529/55A0B7EF" Ref="C67"  Part="1"
 AR Path="/55A5B809/55A0B7EF" Ref="C75"  Part="1"
-F 0 "C75" H 7825 2300 50  0000 L CNN
+F 0 "C67" H 7825 2300 50  0000 L CNN
 F 1 "100n" H 7825 2100 50  0000 L CNN
 F 2 "Capacitors_SMD:C_0805_HandSoldering" H 7838 2050 30  0001 C CNN
@@
 AR Path="/55A0A529/55A0B7F9" Ref="#PWR0167"  Part="1"
 AR Path="/55A5B809/55A0B7F9" Ref="#PWR0181"  Part="1"
-F 0 "#PWR0181" H 7450 2150 50  0001 C CNN
+F 0 "#PWR0167" H 7450 2150 50  0001 C CNN
 F 1 "GNDA" H 7450 2250 50  0000 C CNN
 F 2 "" H 7450 2400 60  0000 C CNN
@@
 AR Path="/55A0A529/55A0B7FF" Ref="#PWR0168"  Part="1"
 AR Path="/55A5B809/55A0B7FF" Ref="#PWR0182"  Part="1"
-F 0 "#PWR0182" H 7350 3000 50  0001 C CNN
+F 0 "#PWR0168" H 7350 3000 50  0001 C CNN
 F 1 "GND" H 7350 3100 50  0000 C CNN
 F 2 "" H 7350 3250 60  0000 C CNN
@@
 AR Path="/55A0A529/55A0D1BD" Ref="#PWR0169"  Part="1"
 AR Path="/55A5B809/55A0D1BD" Ref="#PWR0183"  Part="1"
-F 0 "#PWR0183" H 7700 8500 50  0001 C CNN
+F 0 "#PWR0169" H 7700 8500 50  0001 C CNN
 F 1 "GNDA" H 7700 8600 50  0000 C CNN
 F 2 "" H 7700 8750 60  0000 C CNN
@@
 AR Path="/55A0A529/55A0D66F" Ref="#PWR0170"  Part="1"
 AR Path="/55A5B809/55A0D66F" Ref="#PWR0184"  Part="1"
-F 0 "#PWR0184" H 8000 4200 50  0001 C CNN
+F 0 "#PWR0170" H 8000 4200 50  0001 C CNN
 F 1 "GNDA" H 8000 4300 50  0000 C CNN
 F 2 "" H 8000 4450 60  0000 C CNN
@@
 AR Path="/55A0A529/55BCAD10" Ref="#FLG0171"  Part="1"
 AR Path="/55A5B809/55BCAD10" Ref="#FLG0185"  Part="1"
-F 0 "#FLG0185" H 9450 3345 50  0001 C CNN
+F 0 "#FLG0171" H 9450 3345 50  0001 C CNN
 F 1 "PWR_FLAG" H 9450 3430 50  0000 C CNN
 F 2 "" H 9450 3250 60  0000 C CNN
@@
 AR Path="/55A0A529/55BCAD90" Ref="#FLG0172"  Part="1"
 AR Path="/55A5B809/55BCAD90" Ref="#FLG0186"  Part="1"
-F 0 "#FLG0186" H 9450 4745 50  0001 C CNN
+F 0 "#FLG0172" H 9450 4745 50  0001 C CNN
 F 1 "PWR_FLAG" H 9450 4830 50  0000 C CNN
 F 2 "" H 9450 4650 60  0000 C CNN

Commit message: a
Changed lines of the file:
@@
 $Descr A3 16535 11693
 encoding utf-8
-Sheet 6 7
+Sheet 7 7
 Title ""
 Date ""
@@
 AR Path="/55A0A529/55A0AE22" Ref="U21"  Part="1"
 AR Path="/55A5B809/55A0AE22" Ref="U23"  Part="1"
-F 0 "U21" H 8400 7900 60  0000 C CNN
+F 0 "U23" H 8400 7900 60  0000 C CNN
 F 1 "AD5543" H 8500 8350 60  0000 C CNN
 F 2 "Housings_SOIC:SOIC-8_3.9x4.9mm_Pitch1.27mm" H 7650 8100 60  0001 C CNN
@@
 AR Path="/55A0A529/55A0AE2F" Ref="C64"  Part="1"
 AR Path="/55A5B809/55A0AE2F" Ref="C72"  Part="1"
-F 0 "C64" H 7325 7550 50  0000 L CNN
+F 0 "C72" H 7325 7550 50  0000 L CNN
 F 1 "100n" H 7325 7350 50  0000 L CNN
 F 2 "Capacitors_SMD:C_0805_HandSoldering" H 7338 7300 30  0001 C CNN
@@
 AR Path="/55A0A529/55A0AE38" Ref="#PWR0159"  Part="1"
 AR Path="/55A5B809/55A0AE38" Ref="#PWR0173"  Part="1"
-F 0 "#PWR0159" H 7600 7450 30  0001 C CNN
+F 0 "#PWR0173" H 7600 7450 30  0001 C CNN
 F 1 "VDD" H 7600 7460 30  0000 C CNN
 F 2 "" H 7600 7350 60  0000 C CNN
@@
 AR Path="/55A0A529/55A0AE3F" Ref="U8"  Part="2"
 AR Path="/55A5B809/55A0AE3F" Ref="U9"  Part="2"
-F 0 "U8" H 9750 8100 60  0000 C CNN
+F 0 "U9" H 9750 8100 60  0000 C CNN
 F 1 "AD8672" H 9750 8500 60  0000 C CNN
 F 2 "Housings_SOIC:SOIC-8_3.9x4.9mm_Pitch1.27mm" H 9450 8300 60  0001 C CNN
@@
 AR Path="/55A0A529/55A0AE49" Ref="#PWR0160"  Part="1"
 AR Path="/55A5B809/55A0AE49" Ref="#PWR0174"  Part="1"
-F 0 "#PWR0160" H 8850 8350 50  0001 C CNN
+F 0 "#PWR0174" H 8850 8350 50  0001 C CNN
 F 1 "GNDA" H 8850 8450 50  0000 C CNN
 F 2 "" H 8850 8600 60  0000 C CNN
@@
 AR Path="/55A0A529/55A0AE5A" Ref="C68"  Part="1"
 AR Path="/55A5B809/55A0AE5A" Ref="C76"  Part="1"
-F 0 "C68" H 8825 7900 50  0000 L CNN
+F 0 "C76" H 8825 7900 50  0000 L CNN
 F 1 "1n" H 8825 7700 50  0000 L CNN
 F 2 "Capacitors_SMD:C_0805_HandSoldering" H 8838 7650 30  0001 C CNN
@@
 AR Path="/55A0A529/55A0AE9E" Ref="C65"  Part="1"
 AR Path="/55A5B809/55A0AE9E" Ref="C73"  Part="1"
-F 0 "C65" H 7525 6600 50  0000 L CNN
+F 0 "C73" H 7525 6600 50  0000 L CNN
 F 1 "100n" H 7525 6400 50  0000 L CNN
 F 2 "Capacitors_SMD:C_0805_HandSoldering" H 7538 6350 30  0001 C CNN
@@
 AR Path="/55A0A529/55A0AEA9" Ref="#PWR0161"  Part="1"
 AR Path="/55A5B809/55A0AEA9" Ref="#PWR0175"  Part="1"
-F 0 "#PWR0161" H 7150 6450 50  0001 C CNN
+F 0 "#PWR0175" H 7150 6450 50  0001 C CNN
 F 1 "GNDA" H 7150 6550 50  0000 C CNN
 F 2 "" H 7150 6700 60  0000 C CNN
@@
 AR Path="/55A0A529/55A0AEAF" Ref="#PWR0162"  Part="1"
 AR Path="/55A5B809/55A0AEAF" Ref="#PWR0176"  Part="1"
-F 0 "#PWR0162" H 7050 7300 50  0001 C CNN
+F 0 "#PWR0176" H 7050 7300 50  0001 C CNN
 F 1 "GND" H 7050 7400 50  0000 C CNN
 F 2 "" H 7050 7550 60  0000 C CNN
@@
 AR Path="/55A0A529/55A0B77B" Ref="U22"  Part="1"
 AR Path="/55A5B809/55A0B77B" Ref="U24"  Part="1"
-F 0 "U22" H 8700 3600 60  0000 C CNN
+F 0 "U24" H 8700 3600 60  0000 C CNN
 F 1 "AD5543" H 8800 4050 60  0000 C CNN
 F 2 "Housings_SOIC:SOIC-8_3.9x4.9mm_Pitch1.27mm" H 7950 3800 60  0001 C CNN
@@
 AR Path="/55A0A529/55A0B787" Ref="C66"  Part="1"
 AR Path="/55A5B809/55A0B787" Ref="C74"  Part="1"
-F 0 "C66" H 7625 3250 50  0000 L CNN
+F 0 "C74" H 7625 3250 50  0000 L CNN
 F 1 "100n" H 7625 3050 50  0000 L CNN
 F 2 "Capacitors_SMD:C_0805_HandSoldering" H 7638 3000 30  0001 C CNN
@@
 AR Path="/55A0A529/55A0B78F" Ref="#PWR0163"  Part="1"
 AR Path="/55A5B809/55A0B78F" Ref="#PWR0177"  Part="1"
-F 0 "#PWR0163" H 7900 3150 30  0001 C CNN
+F 0 "#PWR0177" H 7900 3150 30  0001 C CNN
 F 1 "VDD" H 7900 3160 30  0000 C CNN
 F 2 "" H 7900 3050 60  0000 C CNN
@@
 AR Path="/55A0A529/55A0B796" Ref="U8"  Part="1"
 AR Path="/55A5B809/55A0B796" Ref="U9"  Part="1"
-F 0 "U8" H 10050 3800 60  0000 C CNN
+F 0 "U9" H 10050 3800 60  0000 C CNN
 F 1 "AD8672" H 10050 4200 60  0000 C CNN
 F 2 "Housings_SOIC:SOIC-8_3.9x4.9mm_Pitch1.27mm" H 9750 4000 60  0001 C CNN
@@
 AR Path="/55A0A529/55A0B79F" Ref="#PWR0164"  Part="1"
 AR Path="/55A5B809/55A0B79F" Ref="#PWR0178"  Part="1"
-F 0 "#PWR0164" H 9150 4050 50  0001 C CNN
+F 0 "#PWR0178" H 9150 4050 50  0001 C CNN
 F 1 "GNDA" H 9150 4150 50  0000 C CNN
 F 2 "" H 9150 4300 60  0000 C CNN
@@
 AR Path="/55A0A529/55A0B7B0" Ref="C69"  Part="1"
 AR Path="/55A5B809/55A0B7B0" Ref="C77"  Part="1"
-F 0 "C69" H 9125 3600 50  0000 L CNN
+F 0 "C77" H 9125 3600 50  0000 L CNN
 F 1 "1n" H 9125 3400 50  0000 L CNN
 F 2 "Capacitors_SMD:C_0805_HandSoldering" H 9138 3350 30  0001 C CNN
@@
 AR Path="/55A0A529/55A0B7BC" Ref="R67"  Part="1"
 AR Path="/55A5B809/55A0B7BC" Ref="R69"  Part="1"
-F 0 "R67" V 9780 3100 50  0000 C CNN
+F 0 "R69" V 9780 3100 50  0000 C CNN
 F 1 "16 5%" V 9700 3100 50  0000 C CNN
 F 2 "Resistors_SMD:R_0805_HandSoldering" V 9630 3100 30  0001 C CNN
@@
 AR Path="/55A0A529/55A0B7C2" Ref="C70"  Part="1"
 AR Path="/55A5B809/55A0B7C2" Ref="C78"  Part="1"
-F 0 "C70" H 9975 3450 50  0000 L CNN
+F 0 "C78" H 9975 3450 50  0000 L CNN
 F 1 "100n" H 9975 3250 50  0000 L CNN
 F 2 "Capacitors_SMD:C_0805_HandSoldering" H 9988 3200 30  0001 C CNN
@@
 AR Path="/55A0A529/55A0B7CC" Ref="#PWR0165"  Part="1"
 AR Path="/55A5B809/55A0B7CC" Ref="#PWR0179"  Part="1"
-F 0 "#PWR0165" H 10200 3200 50  0001 C CNN
+F 0 "#PWR0179" H 10200 3200 50  0001 C CNN
 F 1 "GNDA" H 10200 3300 50  0000 C CNN
 F 2 "" H 10200 3450 60  0000 C CNN
@@
 AR Path="/55A0A529/55A0B7D5" Ref="R68"  Part="1"
 AR Path="/55A5B809/55A0B7D5" Ref="R70"  Part="1"
-F 0 "R68" V 9780 4800 50  0000 C CNN
+F 0 "R70" V 9780 4800 50  0000 C CNN
 F 1 "16 5%" V 9700 4800 50  0000 C CNN
 F 2 "Resistors_SMD:R_0805_HandSoldering" V 9630 4800 30  0001 C CNN
@@
 AR Path="/55A0A529/55A0B7E0" Ref="C71"  Part="1"
 AR Path="/55A5B809/55A0B7E0" Ref="C79"  Part="1"
-F 0 "C71" H 10025 4900 50  0000 L CNN
+F 0 "C79" H 10025 4900 50  0000 L CNN
 F 1 "100n" H 10025 4700 50  0000 L CNN
 F 2 "Capacitors_SMD:C_0805_HandSoldering" H 10038 4650 30  0001 C CNN
@@
 AR Path="/55A0A529/55A0B7E7" Ref="#PWR0166"  Part="1"
 AR Path="/55A5B809/55A0B7E7" Ref="#PWR0180"  Part="1"
-F 0 "#PWR0166" H 10000 4850 50  0001 C CNN
+F 0 "#PWR0180" H 10000 4850 50  0001 C CNN
 F 1 "GNDA" H 10000 4950 50  0000 C CNN
 F 2 "" H 10000 5100 60  0000 C CNN
@@
 AR Path="/55A0A529/55A0B7EF" Ref="C67"  Part="1"
 AR Path="/55A5B809/55A0B7EF" Ref="C75"  Part="1"
-F 0 "C67" H 7825 2300 50  0000 L CNN
+F 0 "C75" H 7825 2300 50  0000 L CNN
 F 1 "100n" H 7825 2100 50  0000 L CNN
 F 2 "Capacitors_SMD:C_0805_HandSoldering" H 7838 2050 30  0001 C CNN
@@
 AR Path="/55A0A529/55A0B7F9" Ref="#PWR0167"  Part="1"
 AR Path="/55A5B809/55A0B7F9" Ref="#PWR0181"  Part="1"
-F 0 "#PWR0167" H 7450 2150 50  0001 C CNN
+F 0 "#PWR0181" H 7450 2150 50  0001 C CNN
 F 1 "GNDA" H 7450 2250 50  0000 C CNN
 F 2 "" H 7450 2400 60  0000 C CNN
@@
 AR Path="/55A0A529/55A0B7FF" Ref="#PWR0168"  Part="1"
 AR Path="/55A5B809/55A0B7FF" Ref="#PWR0182"  Part="1"
-F 0 "#PWR0168" H 7350 3000 50  0001 C CNN
+F 0 "#PWR0182" H 7350 3000 50  0001 C CNN
 F 1 "GND" H 7350 3100 50  0000 C CNN
 F 2 "" H 7350 3250 60  0000 C CNN
@@
 AR Path="/55A0A529/55A0D1BD" Ref="#PWR0169"  Part="1"
 AR Path="/55A5B809/55A0D1BD" Ref="#PWR0183"  Part="1"
-F 0 "#PWR0169" H 7700 8500 50  0001 C CNN
+F 0 "#PWR0183" H 7700 8500 50  0001 C CNN
 F 1 "GNDA" H 7700 8600 50  0000 C CNN
 F 2 "" H 7700 8750 60  0000 C CNN
@@
 AR Path="/55A0A529/55A0D66F" Ref="#PWR0170"  Part="1"
 AR Path="/55A5B809/55A0D66F" Ref="#PWR0184"  Part="1"
-F 0 "#PWR0170" H 8000 4200 50  0001 C CNN
+F 0 "#PWR0184" H 8000 4200 50  0001 C CNN
 F 1 "GNDA" H 8000 4300 50  0000 C CNN
 F 2 "" H 8000 4450 60  0000 C CNN
@@
 AR Path="/55A0A529/55BCAD10" Ref="#FLG0171"  Part="1"
 AR Path="/55A5B809/55BCAD10" Ref="#FLG0185"  Part="1"
-F 0 "#FLG0171" H 9450 3345 50  0001 C CNN
+F 0 "#FLG0185" H 9450 3345 50  0001 C CNN
 F 1 "PWR_FLAG" H 9450 3430 50  0000 C CNN
 F 2 "" H 9450 3250 60  0000 C CNN
@@
 AR Path="/55A0A529/55BCAD90" Ref="#FLG0172"  Part="1"
 AR Path="/55A5B809/55BCAD90" Ref="#FLG0186"  Part="1"
-F 0 "#FLG0172" H 9450 4745 50  0001 C CNN
+F 0 "#FLG0186" H 9450 4745 50  0001 C CNN
 F 1 "PWR_FLAG" H 9450 4830 50  0000 C CNN
 F 2 "" H 9450 4650 60  0000 C CNN
